File: schematics/main/main.kicad_sch (KiCad schematic)
At the start: 17 parts, among them J1 1602 Display I2C, J2 12V-DC-Jack, J3 Conn_01x02, J4 Conn_01x02, J5 Conn_01x02, J6 Conn_01x02, K1 Relay_SPST-NO, SW1 RotaryEncoder_Switch, SW2 取り消しボタン, SW3 開扉検知用リミットスイッチ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

Commit message: Added firmware and so on
Parts:
- removed SW4: SW_DPST, symbol Switch:SW_DPST
Connections:
- net +12V: now also J2.2
- net GND: now also BZ1.1 (+), J2.1
- net at A1.11 (GPIO8): now also BZ1.2 (-)
Other:
- moved on the sheet: BZ1
Changed lines of the file:
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@@
 	(wire
 		(pts
+			(xy 76.2 119.38) (xy 76.2 109.22)
+		)
+		(stroke
+			(width 0)
+			(type default)
+		)
+	)
+	(wire
+		(pts
 			(xy 27.94 91.44) (xy 99.06 91.44)
 		)
@@
 	(wire
 		(pts
+			(xy 76.2 109.22) (xy 99.06 109.22)
+		)
+		(stroke
+			(width 0)
+			(type default)
+		)
+	)
+	(wire
+		(pts
 			(xy 177.8 115.57) (xy 238.76 115.57)
 		)
@@
 	(wire
 		(pts
-			(xy 233.68 133.35) (xy 257.81 133.35)
+			(xy 76.2 124.46) (xy 76.2 128.27)
 		)
 		(stroke
@@
 	(wire
 		(pts
-			(xy 208.28 36.83) (xy 213.36 36.83)
+			(xy 233.68 133.35) (xy 257.81 133.35)
 		)
 		(stroke
@@
 	(wire
 		(pts
-			(xy 68.58 154.94) (xy 177.8 154.94)
+			(xy 208.28 36.83) (xy 226.06 36.83)
 		)
 		(stroke
@@
 	(wire
 		(pts
-			(xy 254 72.39) (xy 247.65 72.39)
+			(xy 68.58 154.94) (xy 177.8 154.94)
 		)
 		(stroke
@@
 	(wire
 		(pts
-			(xy 60.96 99.06) (xy 99.06 99.06)
+			(xy 254 72.39) (xy 247.65 72.39)
 		)
 		(stroke
@@
 	(wire
 		(pts
-			(xy 223.52 36.83) (xy 226.06 36.83)
+			(xy 60.96 99.06) (xy 99.06 99.06)
 		)
 		(stroke
@@
 	(wire
 		(pts
-			(xy 223.52 41.91) (xy 226.06 41.91)
-		)
-		(stroke
-			(width 0)
-			(type default)
-		)
-	)
-	(wire
-		(pts
 			(xy 34.29 114.3) (xy 44.45 114.3)
 		)
@@
 	(wire
 		(pts
-			(xy 208.28 41.91) (xy 213.36 41.91)
+			(xy 208.28 41.91) (xy 226.06 41.91)
 		)
 		(stroke
@@
 	(symbol
 		(lib_id "power:GND")
+		(at 76.2 128.27 0)
+		(unit 1)
+		(body_style 1)
+		(exclude_from_sim no)
+		(in_bom yes)
+		(on_board yes)
+		(in_pos_files yes)
+		(dnp no)
+		(fields_autoplaced yes)
+		(property "Reference" "#PWR021"
+			(at 76.2 134.62 0)
+			(hide yes)
+			(show_name no)
+			(do_not_autoplace no)
+			(effects
+				(font
+					(size 1.27 1.27)
+				)
+			)
+		)
+		(property "Value" "GND"
+			(at 76.2 133.35 0)
+			(show_name no)
+			(do_not_autoplace no)
+			(effects
+				(font
+					(size 1.27 1.27)
+				)
+			)
+		)
+		(property "Footprint" ""
+			(at 76.2 128.27 0)
+			(hide yes)
+			(show_name no)
+			(do_not_autoplace no)
+			(effects
+				(font
+					(size 1.27 1.27)
+				)
+			)
+		)
+		(property "Datasheet" ""
+			(at 76.2 128.27 0)
+			(hide yes)
+			(show_name no)
+			(do_not_autoplace no)
+			(effects
+				(font
+					(size 1.27 1.27)
+				)
+			)
+		)
+		(property "Description" "Power symbol creates a global label with name \"GND\" , ground"
+			(at 76.2 128.27 0)
+			(hide yes)
+			(show_name no)
+			(do_not_autoplace no)
+			(effects
+				(font
+					(size 1.27 1.27)
+				)
+			)
+		)
+		(pin "1"
+		)
+		(instances
+			(project "main"
+				(path "/572fe60a-408e-4e3f-8200-64ed478fa3a2"
+					(reference "#PWR021")
+					(unit 1)
+				)
+			)
+		)
+	)
+	(symbol
+		(lib_id "power:GND")
 		(at 53.34 121.92 0)
 		(unit 1)
@@
 	(symbol
 		(lib_id "Device:Buzzer")
-		(at 166.37 60.96 0)
+		(at 73.66 121.92 180)
 		(unit 1)
 		(body_style 1)
@@
 		(fields_autoplaced yes)
 		(property "Reference" "BZ1"
-			(at 170.18 59.6899 0)
+			(at 72.9049 114.3 0)
 			(show_name no)
 			(do_not_autoplace no)
@@
 					(size 1.27 1.27)
 				)
-				(justify left)
 			)
 		)
 		(property "Value" "Buzzer"
-			(at 170.18 62.2299 0)
+			(at 72.9049 116.84 0)
 			(show_name no)
 			(do_not_autoplace no)
@@
 					(size 1.27 1.27)
 				)
-				(justify left)
 			)
 		)
 		(property "Footprint" ""
-			(at 165.735 58.42 90)
+			(at 74.295 124.46 90)
 			(hide yes)
 			(show_name no)
@@
 		)
 		(property "Datasheet" ""
-			(at 165.735 58.42 90)
+			(at 74.295 124.46 90)
 			(hide yes)
 			(show_name no)
@@
 		)
 		(property "Description" "Buzzer, polarized"
-			(at 166.37 60.96 0)
+			(at 73.66 121.92 0)
 			(hide yes)
 			(show_name no)
@@
 					(unit 1)
 				)
-			)
-		)
-	)
-	(symbol
-		(lib_id "Switch:SW_DPST")
-		(at 218.44 39.37 0)
-		(unit 1)
-		(body_style 1)
-		(exclude_from_sim no)
-		(in_bom yes)
-		(on_board yes)
-		(in_pos_files yes)
-		(dnp no)
-		(fields_autoplaced yes)
-		(property "Reference" "SW4"
-			(at 218.44 30.48 0)
-			(show_name no)
-			(do_not_autoplace no)
-			(effects
-				(font
-					(size 1.27 1.27)
-				)
-			)
-		)
-		(property "Value" "SW_DPST"
-			(at 218.44 33.02 0)
-			(show_name no)
-			(do_not_autoplace no)
-			(effects
-				(font
-					(size 1.27 1.27)
-				)
-			)
-		)
-		(property "Footprint" ""
-			(at 218.44 39.37 0)
-			(hide yes)
-			(show_name no)
-			(do_not_autoplace no)
-			(effects
-				(font
-					(size 1.27 1.27)
-				)
-			)
-		)
-		(property "Datasheet" ""
-			(at 218.44 39.37 0)
-			(hide yes)
-			(show_name no)
-			(do_not_autoplace no)
-			(effects
-				(font
-					(size 1.27 1.27)
-				)
-			)
-		)
-		(property "Description" "Double Pole Single Throw (DPST) Switch"
-			(at 218.44 39.37 0)
-			(hide yes)
-			(show_name no)
-			(do_not_autoplace no)
-			(effects
-				(font
-					(size 1.27 1.27)
-				)
-			)
-		)
-		(pin "2"
-		)
-		(pin "4"
-		)
-		(pin "1"
-		)
-		(pin "3"
-		)
-		(instances
-			(project "main"
-				(path "/572fe60a-408e-4e3f-8200-64ed478fa3a2"
-					(reference "SW4")
-					(unit 1)
-				)
